File: 4LayerV1/ATSAMA5D27-1G.sch (KiCad schematic (older format))
At the start: 172 parts, among them J1 Conn_01x16, J2 Conn_01x12, J3 USB_B_Micro, J4 Conn_01x02, J5 Conn_01x02, J6 1051620001, J7 USB_B_Micro, Q1 BSS138, Q2 BSS138, Q3 BSS138, Q4 BSS138, Q5 BSS138, U1 ATSAMA5D27C-D1G, U2 ACT8945AQJ305-T, U3 MIC5247-2.0, Y1 NX2012SA_32-768KHz, Y2 NX2016SA_24MHz

Commit message: Move symbols into a local library.
Loading this project into KiCad showed there were missing symbol
libraries. These appear to exist only on the hard drive of the original
author. I have rescued these symbols from the cache file and moved them
into a new local library (with the same name as the project).

I also added a .gitignore to remove all the backup/temp files.
Parts:
- J6: symbol 1051620001:1051620001 -> ATSAMA5D27-1G:1051620001
- PB1: symbol OSD3358-CHIP:MINI_PUSHBUTTON -> ATSAMA5D27-1G:MINI_PUSHBUTTON
- U1: footprint ATSAMA5D27C-D1G-CU:BGA289C80P17X17_1400X1400X120N -> ATSAMA5D27-1G:BGA289C80P17X17_1400X1400X120N; symbol ATSAMA5D27C-D1G-CU:ATSAMA5D27C-D1G -> ATSAMA5D27-1G:ATSAMA5D27C-D1G-CU
- U2: symbol ACT8945AQJ305-T:ACT8945AQJ305-T -> ATSAMA5D27-1G:ACT8945AQJ305-T
- U3: symbol symbols:MIC5247-2.0 -> ATSAMA5D27-1G:MIC5247-2.0
Connections:
- no-connect marks 0 -> 1
Changed lines of the file:
@@
 EESchema Schematic File Version 4
-LIBS:ATSAMA5D27-1G-cache
 EELAYER 30 0
 EELAYER END
@@
 $EndComp
 $Comp
-L ATSAMA5D27C-D1G-CU:ATSAMA5D27C-D1G U1
+L ATSAMA5D27-1G:ATSAMA5D27C-D1G-CU U1
 U 1 1 5B9FFE8B
 P 14100 7950
 F 0 "U1" H 13981 9665 50  0000 C CNN
 F 1 "ATSAMA5D27C-D1G" H 13981 9574 50  0000 C CNN
-F 2 "ATSAMA5D27C-D1G-CU:BGA289C80P17X17_1400X1400X120N" H 14100 7600 50  0001 C CNN
+F 2 "ATSAMA5D27-1G:BGA289C80P17X17_1400X1400X120N" H 14100 7600 50  0001 C CNN
 F 3 "" H 14100 7600 50  0001 C CNN
 	1    14100 7950
@@
 $EndComp
 $Comp
-L ATSAMA5D27C-D1G-CU:ATSAMA5D27C-D1G U1
+L ATSAMA5D27-1G:ATSAMA5D27C-D1G-CU U1
 U 2 1 5B9FFEF8
 P 15650 7950
 F 0 "U1" H 15531 9665 50  0000 C CNN
 F 1 "ATSAMA5D27C-D1G" H 15531 9574 50  0000 C CNN
-F 2 "ATSAMA5D27C-D1G-CU:BGA289C80P17X17_1400X1400X120N" H 15650 7600 50  0001 C CNN
+F 2 "ATSAMA5D27-1G:BGA289C80P17X17_1400X1400X120N" H 15650 7600 50  0001 C CNN
 F 3 "" H 15650 7600 50  0001 C CNN
 	2    15650 7950
@@
 $EndComp
 $Comp
-L ATSAMA5D27C-D1G-CU:ATSAMA5D27C-D1G U1
+L ATSAMA5D27-1G:ATSAMA5D27C-D1G-CU U1
 U 3 1 5B9FFF5B
 P 17300 7950
 F 0 "U1" H 17181 9665 50  0000 C CNN
 F 1 "ATSAMA5D27C-D1G" H 17181 9574 50  0000 C CNN
-F 2 "ATSAMA5D27C-D1G-CU:BGA289C80P17X17_1400X1400X120N" H 17300 7600 50  0001 C CNN
+F 2 "ATSAMA5D27-1G:BGA289C80P17X17_1400X1400X120N" H 17300 7600 50  0001 C CNN
 F 3 "" H 17300 7600 50  0001 C CNN
 	3    17300 7950
@@
 $EndComp
 $Comp
-L ATSAMA5D27C-D1G-CU:ATSAMA5D27C-D1G U1
+L ATSAMA5D27-1G:ATSAMA5D27C-D1G-CU U1
 U 6 1 5BA0005F
 P 17300 3200
 F 0 "U1" H 17275 4615 50  0000 C CNN
 F 1 "ATSAMA5D27C-D1G" H 17275 4524 50  0000 C CNN
-F 2 "ATSAMA5D27C-D1G-CU:BGA289C80P17X17_1400X1400X120N" H 17300 2850 50  0001 C CNN
+F 2 "ATSAMA5D27-1G:BGA289C80P17X17_1400X1400X120N" H 17300 2850 50  0001 C CNN
 F 3 "" H 17300 2850 50  0001 C CNN
 	6    17300 3200
@@
 $EndComp
 $Comp
-L ATSAMA5D27C-D1G-CU:ATSAMA5D27C-D1G U1
+L ATSAMA5D27-1G:ATSAMA5D27C-D1G-CU U1
 U 7 1 5BA00124
 P 7800 2650
 F 0 "U1" H 7800 4365 50  0000 C CNN
 F 1 "ATSAMA5D27C-D1G" H 7800 4274 50  0000 C CNN
-F 2 "ATSAMA5D27C-D1G-CU:BGA289C80P17X17_1400X1400X120N" H 7800 2300 50  0001 C CNN
+F 2 "ATSAMA5D27-1G:BGA289C80P17X17_1400X1400X120N" H 7800 2300 50  0001 C CNN
 F 3 "" H 7800 2300 50  0001 C CNN
 	7    7800 2650
@@
 $EndComp
 $Comp
-L ATSAMA5D27C-D1G-CU:ATSAMA5D27C-D1G U1
+L ATSAMA5D27-1G:ATSAMA5D27C-D1G-CU U1
 U 4 1 5BA004C3
 P 18900 7950
 F 0 "U1" H 18781 9665 50  0000 C CNN
 F 1 "ATSAMA5D27C-D1G" H 18781 9574 50  0000 C CNN
-F 2 "ATSAMA5D27C-D1G-CU:BGA289C80P17X17_1400X1400X120N" H 18900 7600 50  0001 C CNN
+F 2 "ATSAMA5D27-1G:BGA289C80P17X17_1400X1400X120N" H 18900 7600 50  0001 C CNN
 F 3 "" H 18900 7600 50  0001 C CNN
 	4    18900 7950
@@
 $EndComp
 $Comp
-L ACT8945AQJ305-T:ACT8945AQJ305-T U2
+L ATSAMA5D27-1G:ACT8945AQJ305-T U2
 U 1 1 5BA018D2
 P 6300 7950
@@
 $EndComp
 $Comp
-L OSD3358-CHIP:MINI_PUSHBUTTON PB1
+L ATSAMA5D27-1G:MINI_PUSHBUTTON PB1
 U 1 1 5BB34D10
 P 5000 10400
@@
 	10000 13500 10000 13600
 $Comp
-L 1051620001:1051620001 J6
+L ATSAMA5D27-1G:1051620001 J6
 U 1 1 5CABC418
 P 7650 13800
@@
 	3400 15950 3400 15900
 $Comp
-L OSD3358-CHIP:CGND #SUPPLY0104
+L ATSAMA5D27-1G:CGND #SUPPLY0104
 U 1 1 5EB1EFA2
 P 1300 13300
@@
 	5000 9400 5500 9400
 $Comp
-L OSD3358-CHIP:CGND #SUPPLY0101
+L ATSAMA5D27-1G:CGND #SUPPLY0101
 U 1 1 5BF04F3A
 P 7500 14550
@@
 $EndComp
 $Comp
-L OSD3358-CHIP:CGND #SUPPLY0102
+L ATSAMA5D27-1G:CGND #SUPPLY0102
 U 1 1 5BF066A9
 P 9100 14550
@@
 $EndComp
 $Comp
-L OSD3358-CHIP:CGND #SUPPLY0103
+L ATSAMA5D27-1G:CGND #SUPPLY0103
 U 1 1 5BF07B9F
 P 3300 16050
@@
 	4650 15950 4650 15900
 $Comp
-L OSD3358-CHIP:CGND #SUPPLY0105
+L ATSAMA5D27-1G:CGND #SUPPLY0105
 U 1 1 5C5A17AB
 P 4550 16050
@@
 VDD_3V3
 $Comp
-L symbols:MIC5247-2.0 U3
+L ATSAMA5D27-1G:MIC5247-2.0 U3
 U 1 1 5E21569C
 P 2300 1650
@@
 	10500 3450 10400 3450
 $Comp
-L ATSAMA5D27C-D1G-CU:ATSAMA5D27C-D1G U1
+L ATSAMA5D27-1G:ATSAMA5D27C-D1G-CU U1
 U 5 1 5B9FFFF6
 P 11150 3650
 F 0 "U1" H 11150 4765 50  0000 C CNN
 F 1 "ATSAMA5D27C-D1G" H 11150 4674 50  0000 C CNN
-F 2 "ATSAMA5D27C-D1G-CU:BGA289C80P17X17_1400X1400X120N" H 11150 3300 50  0001 C CNN
+F 2 "ATSAMA5D27-1G:BGA289C80P17X17_1400X1400X120N" H 11150 3300 50  0001 C CNN
 F 3 "" H 11150 3300 50  0001 C CNN
 	5    11150 3650
@@
 Text Notes 3000 11750 0    157  ~ 31
 SWDIO
+NoConn ~ 2650 1850
 $EndSCHEMATC

Commit message: Added part numbers to Manufacturer_Part_Number field.
I went with Stackpole RMCF-series resistors and TDK caps, but any
make of jellybean will likely do.
Parts:
- C1, C18, C19, C20, C21, C26, C37, C38, C40, C42, C43, C44, C45, C46, C47, C48, C49, C50, C51, C52, C53, C55, C56, C57, C58, C59, C60, C61, C62, C64, C65, C70, C71, C72, C73, C74, C75, C76, C77, C79, C86, C87, C88, C89, C92, C93, C94, C95: Manufacturer_Name (none) -> TDK; Manufacturer_Part_Number (none) -> CGA2B3X7R1E104K050BB
- C10, C13, C14, C15, C16, C22, C23, C24, C25, C28, C5, C7, C8, C85, C9: Manufacturer_Name (none) -> Samsung; Manufacturer_Part_Number (none) -> CL05A106MP5NUNC
- C100: Manufacturer_Name (none) -> TDK; Manufacturer_Part_Number (none) -> CGA2B2C0G1H100D050BA
- C11, C2, C39, C41, C63, C90, C91: Manufacturer_Name (none) -> TDK; Manufacturer_Part_Number (none) -> C1005X5R1A475K050BC
- C12, C17, C30, C33, C4, C6, C67, C69: Manufacturer_Name (none) -> TDK; Manufacturer_Part_Number (none) -> C1005X5R1E225K050BC
- C27, C29, C31, C32, C34, C36: Manufacturer_Name (none) -> TDK; Manufacturer_Part_Number (none) -> CGA2B2X7R1E103K050BA
- C3: Manufacturer_Name (none) -> TDK; Manufacturer_Part_Number (none) -> CGA2B3X7R1H473K050BB
- C35, C54: Manufacturer_Name (none) -> TDK; Manufacturer_Part_Number (none) -> C1005X5R1E105K050BC
- C96, C97: Manufacturer_Name (none) -> TDK; Manufacturer_Part_Number (none) -> CGA2B2C0G1H080D050BA
- C98, C99: Manufacturer_Name (none) -> TDK; Manufacturer_Part_Number (none) -> CGA2B2C0G1H120J050BA
- D2: Manufacturer_Name (none) -> OSRAM; Manufacturer_Part_Number (none) -> LY L29K-H1K2-26-Z
- D3: Manufacturer_Name (none) -> Diodes Incorporated; Manufacturer_Part_Number (none) -> BAT54C-7-F
- D4: Manufacturer_Name (none) -> OSRAM; Manufacturer_Part_Number (none) -> LO L29K-H2K1-24-Z
- D5: Manufacturer_Name (none) -> OSRAM; Manufacturer_Part_Number (none) -> LG L29K-G2J1-24-Z
- FB1, FB2, FB3, FB4, FB5, FB6, FB7: Manufacturer_Name (none) -> Murata; Manufacturer_Part_Number (none) -> BLM15AG100SH1D
- J3: Manufacturer_Name (none) -> Molex; Manufacturer_Part_Number (none) -> 1050170001
- J4: Manufacturer_Name (none) -> JST; Manufacturer_Part_Number (none) -> S2B-PH-SM4-TB
- J7: Manufacturer_Name (none) -> Amphenol; Manufacturer_Part_Number (none) -> 10104111-0001LF
- L1, L2, L3: Manufacturer_Name (none) -> Taiyo Yuden; Manufacturer_Part_Number (none) -> NR3015T2R2M
- L11, L12, L6: Manufacturer_Name (none) -> TDK; Manufacturer_Part_Number (none) -> MLZ1608N100LT000
- PB1: Manufacturer_Name (none) -> C&K; Manufacturer_Part_Number (none) -> KMR231GLFS
- Q1, Q2, Q3, Q4, Q5: Manufacturer_Name (none) -> ON Semiconductor; Manufacturer_Part_Number (none) -> BSS138
- R1: Manufacturer_Name (none) -> Stackpole; Manufacturer_Part_Number (none) -> RMCF0402FT47K0
- R10: Manufacturer_Name (none) -> Vishay Dale; Manufacturer_Part_Number (none) -> CRCW04022M20FKEDC
- R11: Manufacturer_Name (none) -> Stackpole; Manufacturer_Part_Number (none) -> RMCF0402FT1M50
- R12: Manufacturer_Name (none) -> Stackpole; Manufacturer_Part_Number (none) -> RMCF0402FT2K43
- R14, R16, R18, R22, R5, R6: Manufacturer_Name (none) -> Stackpole; Manufacturer_Part_Number (none) -> RMCF0402FT100K
- R15: Manufacturer_Name (none) -> Stackpole; Manufacturer_Part_Number (none) -> RMCF0402FT49K9
- R17, R21, R23: Manufacturer_Name (none) -> Stackpole; Manufacturer_Part_Number (none) -> RMCF0402FT2R20
- R19, R20, R7, R8: Manufacturer_Name (none) -> Stackpole; Manufacturer_Part_Number (none) -> RMCF0402FT1K50
- R2: Manufacturer_Name (none) -> Stackpole; Manufacturer_Part_Number (none) -> RMCF0402FT1K00
- R24, R25, R27, R4: Manufacturer_Name (none) -> Stackpole; Manufacturer_Part_Number (none) -> RMCF0402FT100R
- R26, R3, R32, R37, R39, R9: Manufacturer_Name (none) -> Stackpole; Manufacturer_Part_Number (none) -> RMCF0402FT10K0
- R29: Manufacturer_Name (none) -> Stackpole; Manufacturer_Part_Number (none) -> RMCF0402FT5K60
- R30, R31, R33, R34: Manufacturer_Name (none) -> Stackpole; Manufacturer_Part_Number (none) -> RMCF0402FT68K0
- R35, R38: Manufacturer_Name (none) -> Stackpole; Manufacturer_Part_Number (none) -> RMCF0402FT330R
- R36: Manufacturer_Name (none) -> Stackpole; Manufacturer_Part_Number (none) -> RMCF0402ZT0R00
- U1: Manufacturer_Name (none) -> Atmel; Manufacturer_Part_Number (none) -> ATSAMA5D27C-D1G-CU
- U2: Manufacturer_Name (none) -> Qorvo; Manufacturer_Part_Number (none) -> ACT8945AQJ305-T
- U3: Manufacturer_Name (none) -> Micrel; Manufacturer_Part_Number (none) -> MIC5247-2.0YM5
- Y1: Manufacturer_Name (none) -> NDK; Manufacturer_Part_Number (none) -> NX2012SA-32.768K-STD-MUB-1
- Y2: Manufacturer_Name (none) -> NDK; Manufacturer_Part_Number (none) -> NX2016SA-24MHZ-EXS00A-CS11335
